Commit message: add comments

File: urdf/xacro/mbot_base_gazebo.xacro (robot description, xacro)
@@ -1,18 +1,23 @@
 <?xml version="1.0"?>
 <robot name="mbot" xmlns:xacro="http://www.ros.org/wiki/xacro">
-    <!-- PROPERTY LIST -->
+    <!-- base -->
     <xacro:property name="M_PI" value="3.1415926"/>
     <xacro:property name="base_mass"   value="20" />
-    <xacro:property name="base_radius" value="0.20"/>
-    <xacro:property name="base_length" value="0.16"/>
+    <xacro:property name="base_radius" value="0.15"/>
+    <xacro:property name="base_length" value="0.05"/>
+    <xacro:property name="base_width" value="0.3"/>
+    <xacro:property name="base_leng" value="0.3"/>
+    <xacro:property name="base_higth" value="0.05"/>
+ 	<!-- wheel -->
     <xacro:property name="wheel_mass"   value="2" />
-    <xacro:property name="wheel_radius" value="0.06"/>
-    <xacro:property name="wheel_length" value="0.025"/>
-    <xacro:property name="wheel_joint_y" value="0.19"/>
-    <xacro:property name="wheel_joint_z" value="0.05"/>
+    <xacro:property name="wheel_radius" value="0.025"/>
+    <xacro:property name="wheel_length" value="0.015"/>
+    <xacro:property name="wheel_joint_y" value="0.15"/>
+    <xacro:property name="wheel_joint_z" value="0.02"/>
+	<!-- caster -->
     <xacro:property name="caster_mass"    value="0.5" />
-    <xacro:property name="caster_radius"  value="0.015"/> <!-- wheel_radius - ( base_length/2 - wheel_joint_z) -->
-    <xacro:property name="caster_joint_x" value="0.18"/>
-    <!-- Defining the colors used in this robot -->
+    <xacro:property name="caster_radius"  value="0.01"/> <!-- wheel_radius - ( base_length/2 - wheel_joint_z) -->
+    <xacro:property name="caster_joint_x" value="0.14"/>
+    <!-- colors -->
     <material name="yellow">
         <color rgba="1 0.4 0 1"/>
@@ -40,4 +45,12 @@
                 izz="${m*r*r/2}" />
         </inertial>
+    </xacro:macro>
+    <xacro:macro name="box_inertial_matrix" params="m a b c">
+       <inertial>
+          <mass value="${m}" />
+           <inertia ixx="${m*(b*b+c*c)/12}" ixy = "0" ixz = "0"
+              iyy="${m*(c*c+a*a)/12}" iyz = "0"
+              izz="${m*(a*a+b*b)/12}" />
+       </inertial>
     </xacro:macro>
     <!-- Macro for robot wheel -->
@@ -68,4 +81,5 @@
             <material>Gazebo/Gray</material>
         </gazebo>
+ 		<!-- Transmission is important to link the joints and the controller -->
         <transmission name="${prefix}_wheel_joint_trans">
             <type>transmission_interface/SimpleTransmission</type>
@@ -103,8 +117,10 @@
             <sphere_inertial_matrix  m="${caster_mass}" r="${caster_radius}" />
         </link>
+    	<!-- Add gazebo tag to link -->
         <gazebo reference="${prefix}_caster_link">
-            <material>Gazebo/Black</material>
+            <material>Gazebo/Gray</material>
         </gazebo>
     </xacro:macro>
+    <!-- Macro for robot base -->
     <xacro:macro name="mbot_base_gazebo">
         <link name="base_footprint">
@@ -129,4 +145,5 @@
                 <geometry>
                     <cylinder length="${base_length}" radius="${base_radius}"/>
+                    <!--box size="0.3 0.3 0.05" /-->
                 </geometry>
                 <material name="yellow" />
@@ -136,8 +153,11 @@
                 <geometry>
                     <cylinder length="${base_length}" radius="${base_radius}"/>
+                    <!--box size="0.3 0.3 0.05" /-->
                 </geometry>
             </collision>
             <cylinder_inertial_matrix  m="${base_mass}" r="${base_radius}" h="${base_length}" />
+            <!-- box_inertial_matrix  m="${base_mass}" a="0.3" b="0.3" c="0.05"/-->
         </link>
+    	<!-- Add gazebo tag to link -->
         <gazebo reference="base_link">
             <material>Gazebo/Blue</material>

File: urdf/xacro/mbot_camera_gazebo.xacro (robot description, xacro)
@@ -14,5 +14,5 @@
                 <origin xyz=" 0 0 0 " rpy="0 0 0" />
                 <geometry>
-                    <box size="0.01 0.02 0.06" />
+                    <box size="0.005 0.09 0.02" />
                 </geometry>
                 <material name="black"/>
@@ -21,5 +21,5 @@
                 <origin xyz="0.0 0.0 0.0" rpy="0 0 0" />
                 <geometry>
-                    <box size="0.01 0.04 0.04" />
+                    <box size="0.005 0.09 0.02" />
                 </geometry>
             </collision>

File: urdf/xacro/mbot_gazebo.xacro (robot description, xacro)
@@ -5,13 +5,13 @@
     <xacro:include filename="$(find mbot_sim)/urdf/xacro/mbot_lidar_gazebo.xacro" />
     <xacro:include filename="$(find mbot_sim)/urdf/xacro/mbot_imu_gazebo.xacro" />
-    <xacro:property name="camera_offset_x" value="0.17" />
+    <xacro:property name="camera_offset_x" value="0.13" />
     <xacro:property name="camera_offset_y" value="0" />
-    <xacro:property name="camera_offset_z" value="0.10" />
+    <xacro:property name="camera_offset_z" value="0.035" />
     <xacro:property name="lidar_offset_x" value="0" />
     <xacro:property name="lidar_offset_y" value="0" />
-    <xacro:property name="lidar_offset_z" value="0.105" />
+    <xacro:property name="lidar_offset_z" value="0.06" />
     <xacro:property name="imu_offset_x" value="0" />
     <xacro:property name="imu_offset_y" value="0" />
-    <xacro:property name="imu_offset_z" value="0.6" />
+    <xacro:property name="imu_offset_z" value="0.04" />
     <xacro:mbot_base_gazebo />
     <!-- Camera -->

File: urdf/xacro/mbot_imu_gazebo.xacro (robot description, xacro)
@@ -1,6 +1,4 @@
 <?xml version="1.0"?>
 <robot name="imu" xmlns:xacro="http://www.ros.org/wiki/xacro">
-    <xacro:property name="imu_size"     value="0.1" />
-    <xacro:property name="imu_hight"    value="0.1" />
     <xacro:macro name="use_imu" params="prefix:=imu">
         <link name="${prefix}_link">
@@ -15,12 +13,12 @@
                 <origin xyz="0 0 0" rpy="0 0 0" />
                 <geometry>
-                    <box size="${imu_size} ${imu_size} ${imu_hight}"/>
+                    <cylinder length="0.02" radius="0.045"/>
                 </geometry>
-                <material name="red"/>
+                <material name="black"/>
             </visual>
             <collision>
                 <origin xyz="0.0 0.0 0.0" rpy="0 0 0" />
                 <geometry>
-                    <box size="${imu_size} ${imu_size} ${imu_hight}"/>
+                    <cylinder length="0.02" radius="0.045"/>
                 </geometry>
             </collision>

File: urdf/xacro/mbot_lidar_gazebo.xacro (robot description, xacro)
@@ -13,5 +13,5 @@
                 <origin xyz=" 0 0 0 " rpy="0 0 0" />
                 <geometry>
-                    <cylinder length="0.05" radius="0.05"/>
+                    <cylinder length="0.03" radius="0.030"/>
                 </geometry>
                 <material name="black"/>
@@ -20,5 +20,5 @@
                 <origin xyz="0.0 0.0 0.0" rpy="0 0 0" />
                 <geometry>
-                    <cylinder length="0.06" radius="0.05"/>
+                    <cylinder length="0.03" radius="0.030"/>
                 </geometry>
             </collision>

Commit message: add teleop

File: urdf/xacro/mbot_base_gazebo.xacro (robot description, xacro)
@@ -1,4 +1,4 @@
 <?xml version="1.0"?>
-<robot name="mbot" xmlns:xacro="http://www.ros.org/wiki/xacro">
+<robot name="base" xmlns:xacro="http://www.ros.org/wiki/xacro">
     <!-- base -->
     <xacro:property name="M_PI" value="3.1415926"/>
@@ -21,8 +21,8 @@
     <!-- colors -->
     <material name="yellow">
-        <color rgba="1 0.4 0 1"/>
+        <color rgba="0 0 1 1"/>
     </material>
     <material name="black">
-        <color rgba="0 0 0 0.95"/>
+        <color rgba="0 0 0 1"/>
     </material>
     <material name="gray">
@@ -186,5 +186,5 @@
                 <wheelTorque>30</wheelTorque>
                 <wheelAcceleration>1.8</wheelAcceleration>
-                <commandTopic>cmd_vel</commandTopic>
+                <commandTopic>mbot2/cmd_vel</commandTopic>
                 <odometryFrame>odom</odometryFrame>
                 <odometryTopic>odom</odometryTopic>

File: urdf/xacro/mbot_base_rviz.xacro (robot description, xacro)
@@ -15,8 +15,8 @@
 <!-- Defining the colors used in this robot -->
     <material name="yellow">
-        <color rgba="1 0.4 0 1"/>
+        <color rgba="0 0 1 1"/>
     </material>
     <material name="black">
-        <color rgba="0 0 0 0.95"/>
+        <color rgba="0 0 0 1"/>
     </material>
     <material name="gray">

File: urdf/xacro/mbot_camera_gazebo.xacro (robot description, xacro)
@@ -2,5 +2,5 @@
 <robot name="camera" xmlns:xacro="http://www.ros.org/wiki/xacro">
     <xacro:macro name="use_camera" params="prefix:=camera">
-        <!-- Create laser reference frame -->
+        <!-- Create reference frame -->
         <link name="${prefix}_link">
             <inertial>

File: urdf/xacro/mbot_gazebo.xacro (robot description, xacro)
@@ -15,5 +15,5 @@
     <xacro:property name="imu_offset_z" value="0.04" />
     <xacro:mbot_base_gazebo />
-    <!-- Camera -->
+    <!-- camera -->
     <joint name="camera_joint" type="fixed">
         <origin xyz="${camera_offset_x} ${camera_offset_y} ${camera_offset_z}" rpy="0 0 0" />
@@ -25,5 +25,5 @@
         <origin xyz="${lidar_offset_x} ${lidar_offset_y} ${lidar_offset_z}" rpy="0 0 0" />
         <parent link="base_link"/>
-        <child link="lidar_link"/>
+        <child link="laser_link"/>
     </joint>
     <!-- imu -->
@@ -34,5 +34,5 @@
     </joint>
     <xacro:use_camera prefix="camera"/>
-    <xacro:use_lidar prefix="lidar"/>
+    <xacro:use_laser prefix="laser"/>
     <xacro:use_imu prefix="imu"/>
 </robot>

File: urdf/xacro/mbot_imu_gazebo.xacro (robot description, xacro)
@@ -13,5 +13,5 @@
                 <origin xyz="0 0 0" rpy="0 0 0" />
                 <geometry>
-                    <cylinder length="0.02" radius="0.045"/>
+                    <cylinder length="0.03" radius="0.045"/>
                 </geometry>
                 <material name="black"/>
@@ -20,5 +20,5 @@
                 <origin xyz="0.0 0.0 0.0" rpy="0 0 0" />
                 <geometry>
-                    <cylinder length="0.02" radius="0.045"/>
+                    <cylinder length="0.03" radius="0.045"/>
                 </geometry>
             </collision>
@@ -29,5 +29,5 @@
         <gazebo reference="${prefix}_link">
             <gravity>true</gravity>
-            <sensor type="imu" name="imu_sensor" >
+            <sensor type="imu" name="imu_node" >
                 <always_on>true</always_on>
                 <update_rate>100</update_rate>

File: urdf/xacro/mbot_lidar_gazebo.xacro (robot description, xacro)
@@ -1,5 +1,5 @@
 <?xml version="1.0"?>
-<robot xmlns:xacro="http://www.ros.org/wiki/xacro" name="laser">
-	<xacro:macro name="use_lidar" params="prefix:=lidar">
+<robot name="laser" xmlns:xacro="http://www.ros.org/wiki/xacro" >
+	<xacro:macro name="use_laser" params="prefix:=laser">
         <link name="${prefix}_link">
             <inertial>
@@ -11,5 +11,5 @@
             </inertial>
             <visual>
-                <origin xyz=" 0 0 0 " rpy="0 0 0" />
+                <origin xyz="0 0 0" rpy="0 0 0" />
                 <geometry>
                     <cylinder length="0.03" radius="0.030"/>
@@ -28,5 +28,5 @@
         </gazebo>
         <gazebo reference="${prefix}_link">
-            <sensor type="ray" name="rplidar">
+            <sensor type="ray" name="laser_node">
                 <pose>0 0 0 0 0 0</pose>
                 <visualize>false</visualize>

Commit message: add slam

File: urdf/xacro/mbot_base_gazebo.xacro (robot description, xacro)
@@ -186,5 +186,5 @@
                 <wheelTorque>30</wheelTorque>
                 <wheelAcceleration>1.8</wheelAcceleration>
-                <commandTopic>mbot2/cmd_vel</commandTopic>
+                <commandTopic>cmd_vel</commandTopic>
                 <odometryFrame>odom</odometryFrame>
                 <odometryTopic>odom</odometryTopic>

File: urdf/xacro/mbot_gazebo.xacro (robot description, xacro)
@@ -2,8 +2,8 @@
 <robot name="mbot" xmlns:xacro="http://www.ros.org/wiki/xacro">
     <xacro:include filename="$(find mbot_sim)/urdf/xacro/mbot_base_gazebo.xacro" />
-    <xacro:include filename="$(find mbot_sim)/urdf/xacro/mbot_camera_gazebo.xacro" />
+    <!--xacro:include filename="$(find mbot_sim)/urdf/xacro/mbot_camera_gazebo.xacro" />
     <xacro:include filename="$(find mbot_sim)/urdf/xacro/mbot_lidar_gazebo.xacro" />
-    <xacro:include filename="$(find mbot_sim)/urdf/xacro/mbot_imu_gazebo.xacro" />
-    <xacro:property name="camera_offset_x" value="0.13" />
+    <xacro:include filename="$(find mbot_sim)/urdf/xacro/mbot_imu_gazebo.xacro" /-->
+    <!--xacro:property name="camera_offset_x" value="0.13" />
     <xacro:property name="camera_offset_y" value="0" />
     <xacro:property name="camera_offset_z" value="0.035" />
@@ -13,19 +13,19 @@
     <xacro:property name="imu_offset_x" value="0" />
     <xacro:property name="imu_offset_y" value="0" />
-    <xacro:property name="imu_offset_z" value="0.04" />
+    <xacro:property name="imu_offset_z" value="0.04" /-->
     <xacro:mbot_base_gazebo />
-    <!-- camera -->
+    <!-- camera >
     <joint name="camera_joint" type="fixed">
         <origin xyz="${camera_offset_x} ${camera_offset_y} ${camera_offset_z}" rpy="0 0 0" />
         <parent link="base_link"/>
         <child link="camera_link"/>
-    </joint>
-    <!-- lidar -->
+    </joint-->
+    <!-- lidar >
     <joint name="lidar_joint" type="fixed">
         <origin xyz="${lidar_offset_x} ${lidar_offset_y} ${lidar_offset_z}" rpy="0 0 0" />
         <parent link="base_link"/>
         <child link="laser_link"/>
-    </joint>
-    <!-- imu -->
+    </joint-->
+    <!-- imu >
     <joint name="imu_joint" type="fixed">
         <origin xyz="${imu_offset_x} ${imu_offset_y} ${imu_offset_z}" rpy="0 0 0" />
@@ -35,4 +35,4 @@
     <xacro:use_camera prefix="camera"/>
     <xacro:use_laser prefix="laser"/>
-    <xacro:use_imu prefix="imu"/>
+    <xacro:use_imu prefix="imu"/-->
 </robot>

Commit message: add follow

File: urdf/xacro/mbot_base_gazebo.xacro (robot description, xacro)
@@ -186,5 +186,5 @@
                 <wheelTorque>30</wheelTorque>
                 <wheelAcceleration>1.8</wheelAcceleration>
-                <commandTopic>cmd_vel</commandTopic>
+                <commandTopic>/mbot/cmd_vel</commandTopic>
                 <odometryFrame>odom</odometryFrame>
                 <odometryTopic>odom</odometryTopic>

File: urdf/xacro/mbot_gazebo.xacro (robot description, xacro)
@@ -2,8 +2,8 @@
 <robot name="mbot" xmlns:xacro="http://www.ros.org/wiki/xacro">
     <xacro:include filename="$(find mbot_sim)/urdf/xacro/mbot_base_gazebo.xacro" />
-    <!--xacro:include filename="$(find mbot_sim)/urdf/xacro/mbot_camera_gazebo.xacro" />
+    <xacro:include filename="$(find mbot_sim)/urdf/xacro/mbot_camera_gazebo.xacro" />
     <xacro:include filename="$(find mbot_sim)/urdf/xacro/mbot_lidar_gazebo.xacro" />
-    <xacro:include filename="$(find mbot_sim)/urdf/xacro/mbot_imu_gazebo.xacro" /-->
-    <!--xacro:property name="camera_offset_x" value="0.13" />
+    <xacro:include filename="$(find mbot_sim)/urdf/xacro/mbot_imu_gazebo.xacro" />
+    <xacro:property name="camera_offset_x" value="0.13" />
     <xacro:property name="camera_offset_y" value="0" />
     <xacro:property name="camera_offset_z" value="0.035" />
@@ -13,19 +13,19 @@
     <xacro:property name="imu_offset_x" value="0" />
     <xacro:property name="imu_offset_y" value="0" />
-    <xacro:property name="imu_offset_z" value="0.04" /-->
+    <xacro:property name="imu_offset_z" value="0.04" />
     <xacro:mbot_base_gazebo />
-    <!-- camera >
+    <!-- camera -->
     <joint name="camera_joint" type="fixed">
         <origin xyz="${camera_offset_x} ${camera_offset_y} ${camera_offset_z}" rpy="0 0 0" />
         <parent link="base_link"/>
         <child link="camera_link"/>
-    </joint-->
-    <!-- lidar >
+    </joint>
+    <!-- lidar -->
     <joint name="lidar_joint" type="fixed">
         <origin xyz="${lidar_offset_x} ${lidar_offset_y} ${lidar_offset_z}" rpy="0 0 0" />
         <parent link="base_link"/>
         <child link="laser_link"/>
-    </joint-->
-    <!-- imu >
+    </joint>
+    <!-- imu -->
     <joint name="imu_joint" type="fixed">
         <origin xyz="${imu_offset_x} ${imu_offset_y} ${imu_offset_z}" rpy="0 0 0" />
@@ -35,4 +35,4 @@
     <xacro:use_camera prefix="camera"/>
     <xacro:use_laser prefix="laser"/>
-    <xacro:use_imu prefix="imu"/-->
+    <xacro:use_imu prefix="imu"/>
 </robot>
